File: nsm4202A_MAN3910.kicad_sch (KiCad schematic)
At the start: 19 parts, among them IC1 IS31FL3730-QFLS2-TR, IC2 IS31FL3730-QFLS2-TR, J1 Conn_01x07_Pin, J2 Conn_01x02_Pin, J3 Conn_01x03_Pin

Commit message: Start trace
Connections:
- net +5V: now also J1.4 (Pin_4)
- net D1_C8: now also J1.7 (Pin_7)
- net D1_R1: now also J3.1 (Pin_1)
- net D1_R2: now also J3.2 (Pin_2)
- net D1_R3: now also J3.3 (Pin_3)
- net D1_R4: now also J2.1 (Pin_1)
- net D1_R5: now also J2.2 (Pin_2)
- net GND: now also J1.6 (Pin_6)
- net SDA: now reaches IC1.1 (SDA), R2.2
- net SDA: now also IC2.1 (SDA), J1.2 (Pin_2)
- net SCL: now reaches IC1.2 (SCL), R1.2
- net SCL: now also IC2.2 (SCL), IC2.6 (AD), J1.3 (Pin_3)
- no-connect marks 8 -> 9

Commit message: Updates
Parts:
- removed C2, C5, C6: 100nF, Capacitor_SMD:C_0603_1608Metric_Pad1.08x0.95mm_HandSolder, symbol Device:C
